File: MM26/MM26.kicad_pcb (KiCad board)
At the start: 2 copper layers, 2 parts, among them U1 AZ1117IH-3.3TRG1

Commit message: Imported Everything
Parts:
- removed D1: LED, LED_THT:LED_D2.0mm_W4.8mm_H2.5mm_FlatTop
- added J1: B2B-PH-K-S, B2B_PH_K_S:JST_B2B-PH-K-S, F.Cu at (126.0, 135.9)
- added J2: B2B-PH-K-S, B2B_PH_K_S:JST_B2B-PH-K-S, F.Cu at (126.0, 142.6)
- added J3: Conn_01x06_Pin, Connector_JST:JST_SH_BM06B-SRSS-TB_1x06-1MP_P1.00mm_Vertical, F.Cu at (135.1, 136.0)
- added J4: Conn_01x06_Pin, Connector_JST:JST_SH_BM06B-SRSS-TB_1x06-1MP_P1.00mm_Vertical, F.Cu at (135.1, 142.2)
- added J5: Conn_01x03_Pin, Connector_PinSocket_2.54mm:PinSocket_1x03_P2.54mm_Horizontal, F.Cu at (164.3, 94.6)
- added J6: Conn_01x03_Pin, Connector_PinSocket_2.54mm:PinSocket_1x03_P2.54mm_Horizontal, F.Cu at (164.3, 104.3)
- added J7: Conn_01x03_Pin, Connector_PinSocket_2.54mm:PinSocket_1x03_P2.54mm_Horizontal, F.Cu at (181.5, 120.6)
- added J8: Conn_01x03_Pin, Connector_PinSocket_2.54mm:PinSocket_1x03_P2.54mm_Horizontal, F.Cu at (164.3, 123.7)
- added J9: Conn_01x03_Pin, Connector_PinSocket_2.54mm:PinSocket_1x03_P2.54mm_Horizontal, F.Cu at (164.3, 133.4)
- added SW1: CL-SB-12A-01T, CL_SB_12A_01T:CL-SB-12A-01T_NDC, F.Cu at (173.9, 109.8)
- added U2: NUCLEO-L476RG, NUCLEO-L476RG:MODULE_NUCLEO-L476RG, F.Cu at (86.5, 114.3)
- added U3: ISM330DHCX, Adafruit_ISM330DHCX:ISM330DHCX, F.Cu at (125.3, 109.5)
- added U4: SSD1306, Adafruit_SSD1306:SSD1306, F.Cu at (134.3, 88.3)
- added U5: L293DD, L293DD:SOIC127P1032X265-20N, F.Cu at (173.5, 99.5)
- moved U1 67.6 mm to (135.5, 149.4)
Connections:
- U1 pad 1: unconnected-(U1-GND-Pad1) -> GND
- U1 pad 2: unconnected-(U1-OUTPUT-Pad2) -> VCC
Routing:
- net VCC: track 12.2 -> 0.00 mm

Commit message: all components placed on pcb
just need to route it now
Parts:
- added C1: 10uF, Capacitor_SMD:C_0805_2012Metric_Pad1.18x1.45mm_HandSolder, F.Cu at (234.1, 165.7)
- added C2: 22uF, Capacitor_SMD:C_0805_2012Metric_Pad1.18x1.45mm_HandSolder, F.Cu at (231.1, 165.7)
- added C3: 4.7uF, Capacitor_SMD:C_0805_2012Metric_Pad1.18x1.45mm_HandSolder, F.Cu at (228.1, 165.7)
- added C4: 100nF, Capacitor_SMD:C_0805_2012Metric_Pad1.18x1.45mm_HandSolder, F.Cu at (225.1, 165.7)
- added C5: 4.7uF, Capacitor_SMD:C_0805_2012Metric_Pad1.18x1.45mm_HandSolder, F.Cu at (222.1, 165.7)
- added C6: 10uF, Capacitor_SMD:C_0805_2012Metric_Pad1.18x1.45mm_HandSolder, F.Cu at (219.1, 165.7)
- added H1: MountingHole, MountingHole:MountingHole_2.5mm, F.Cu at (229.0, 214.0)
- added H2: MountingHole, MountingHole:MountingHole_2.5mm, F.Cu at (262.3, 230.4)
- added H3: MountingHole, MountingHole:MountingHole_2.5mm, F.Cu at (244.3, 230.4)
- added H4: MountingHole, MountingHole:MountingHole_2.5mm, F.Cu at (244.3, 162.3)
- added H5: MountingHole, MountingHole:MountingHole_2.5mm, F.Cu at (229.0, 178.7)
- added H6: MountingHole, MountingHole:MountingHole_2.5mm, F.Cu at (262.3, 162.3)
- added H7: MountingHole, MountingHole:MountingHole_2mm, F.Cu at (381.7, 189.0)
- added H8: MountingHole, MountingHole:MountingHole_2mm, F.Cu at (381.7, 203.7)
- added R1: 10k, Resistor_SMD:R_0805_2012Metric_Pad1.20x1.40mm_HandSolder, F.Cu at (234.1, 170.4)
- moved U3 265.9 mm to (373.8, 204.0), turned to -90 degrees
- moved J5 253.2 mm to (395.0, 199.1), turned to 180 degrees
- moved U4 253.1 mm to (366.5, 189.1), turned to 90 degrees
- moved J8 239.6 mm to (385.2, 216.5), turned to 135 degrees
- moved U2 236.6 mm to (308.3, 196.5), turned to -90 degrees
- moved J6 233.5 mm to (366.0, 221.8), turned to 90 degrees
- moved J9 230.1 mm to (389.5, 180.5), turned to -135 degrees
- moved J7 196.4 mm to (371.2, 171.6), turned to -90 degrees
- moved J3 150.0 mm to (262.3, 215.6), turned to -90 degrees
- moved SW1 138.4 mm to (234.4, 234.3)
- moved J1 137.5 mm to (226.4, 229.8), turned to -90 degrees
- moved J4 132.8 mm to (262.4, 180.2), turned to -90 degrees
- moved J2 128.1 mm to (219.8, 229.8), turned to -90 degrees
- moved U5 126.0 mm to (252.2, 197.9), turned to -90 degrees
- moved U1 124.0 mm to (237.2, 220.4)
Connections:
- J3 pad 1: unconnected-(J3-Pin_1-Pad1) -> /M+1
- J3 pad 2: unconnected-(J3-Pin_2-Pad2) -> /M-1
- J3 pad 3: unconnected-(J3-Pin_3-Pad3) -> VCC
- J3 pad 4: unconnected-(J3-Pin_4-Pad4) -> /ENC1_A
- J3 pad 5: unconnected-(J3-Pin_5-Pad5) -> /ENC1_B
- J3 pad 6: unconnected-(J3-Pin_6-Pad6) -> GND
- J4 pad 1: unconnected-(J4-Pin_1-Pad1) -> /M+2
- J4 pad 2: unconnected-(J4-Pin_2-Pad2) -> /M-2
- J4 pad 3: unconnected-(J4-Pin_3-Pad3) -> VCC
- J4 pad 4: unconnected-(J4-Pin_4-Pad4) -> /ENC2_A
- J4 pad 5: unconnected-(J4-Pin_5-Pad5) -> /ENC2_B
- J4 pad 6: unconnected-(J4-Pin_6-Pad6) -> GND
- J5 pad 1: unconnected-(J5-Pin_1-Pad1) -> /IR_OUT_1
- J6 pad 1: unconnected-(J6-Pin_1-Pad1) -> /IR_OUT_4
- J7 pad 1: unconnected-(J7-Pin_1-Pad1) -> /IR_OUT_2
- J8 pad 1: unconnected-(J8-Pin_1-Pad1) -> /IR_OUT_5
- J9 pad 1: unconnected-(J9-Pin_1-Pad1) -> /IR_OUT_3
- U2 pad CN10_13: unconnected-(U2B-PA6-PadCN10_13) -> /ENC2_B
- U2 pad CN10_14: unconnected-(U2B-PA11-PadCN10_14) -> /M1_C
- U2 pad CN10_15: unconnected-(U2B-PA7-PadCN10_15) -> /ENC2_A
- U2 pad CN10_16: unconnected-(U2B-PB12-PadCN10_16) -> /OLED_CS
- U2 pad CN10_21: unconnected-(U2B-PA9-PadCN10_21) -> /M2_C
- U2 pad CN10_22: unconnected-(U2B-PB2-PadCN10_22) -> /IR_OUT_2
- U2 pad CN10_23: unconnected-(U2B-PA8-PadCN10_23) -> /M2_CC
- U2 pad CN10_24: unconnected-(U2B-PB1-PadCN10_24) -> /IR_OUT_1
- U2 pad CN10_26: unconnected-(U2B-PB15-PadCN10_26) -> /IR_OUT_3
- U2 pad CN10_28: unconnected-(U2B-PB14-PadCN10_28) -> /IR_OUT_4
- U2 pad CN10_30: unconnected-(U2B-PB13-PadCN10_30) -> /OLED_SCL
- U2 pad CN10_33: unconnected-(U2B-PA10-PadCN10_33) -> /M1_CC
- U2 pad CN10_34: unconnected-(U2B-PC4-PadCN10_34) -> /IR_OUT_5
- U2 pad CN7_1: unconnected-(U2A-PC10-PadCN7_1) -> /Gyro_SCL
- U2 pad CN7_16: unconnected-(U2A-+3V3-PadCN7_16) -> VCC
- U2 pad CN7_2: unconnected-(U2A-PC11-PadCN7_2) -> /Gyro_MISO
- U2 pad CN7_28: unconnected-(U2A-PA0-PadCN7_28) -> /ENC1_A
- U2 pad CN7_3: unconnected-(U2A-PC12-PadCN7_3) -> /Gyro_MOSI
- U2 pad CN7_30: unconnected-(U2A-PA1-PadCN7_30) -> /ENC1_B
- U2 pad CN7_32: unconnected-(U2A-PA4-PadCN7_32) -> /Gyro_CS
- U2 pad CN7_35: unconnected-(U2A-PC2-PadCN7_35) -> /OLED_MISO
- U2 pad CN7_37: unconnected-(U2A-PC3-PadCN7_37) -> /OLED_MOSI
- U2 pad CN7_5: unconnected-(U2A-VDD-PadCN7_5) -> GND
- U3 pad 1: unconnected-(U3-Vin-Pad1) -> VCC
- U3 pad 14: unconnected-(U3-GND-Pad14) -> GND
- U3 pad 3: unconnected-(U3-GND-Pad3) -> GND
- U3 pad 4: unconnected-(U3-SCL-Pad4) -> /Gyro_SCL
- U3 pad 5: unconnected-(U3-SDA/MOSI-Pad5) -> /Gyro_MOSI
- U3 pad 6: unconnected-(U3-MISO-Pad6) -> /Gyro_MISO
- U3 pad 7: unconnected-(U3-CS-Pad7) -> /Gyro_CS
- U4 pad 1: unconnected-(U4-CS-Pad1) -> /OLED_CS
- U4 pad 3: unconnected-(U4-D/C-Pad3) -> /OLED_MISO
- U4 pad 4: unconnected-(U4-CLK-Pad4) -> /OLED_SCL
- U4 pad 5: unconnected-(U4-DATA-Pad5) -> /OLED_MOSI
- U4 pad 6: unconnected-(U4-VIN-Pad6) -> VCC
- U4 pad 8: unconnected-(U4-GND-Pad8) -> GND
- U5 pad 1: unconnected-(U5-ENABLE_1-Pad1) -> VCC
- U5 pad 10: unconnected-(U5-VS-Pad10) -> VCC
- U5 pad 11: unconnected-(U5-ENABLE_2-Pad11) -> VCC
- U5 pad 12: unconnected-(U5-INPUT_3-Pad12) -> /M2_C
- U5 pad 13: unconnected-(U5-OUTPUT_3-Pad13) -> /M+2
- U5 pad 14: unconnected-(U5-GND__4-Pad14) -> GND
- U5 pad 15: unconnected-(U5-GND__5-Pad15) -> GND
- U5 pad 16: unconnected-(U5-GND__6-Pad16) -> GND
- U5 pad 17: unconnected-(U5-GND__7-Pad17) -> GND
- U5 pad 18: unconnected-(U5-OUTPUT_4-Pad18) -> /M-2
- U5 pad 19: unconnected-(U5-INPUT_4-Pad19) -> /M2_CC
- U5 pad 2: unconnected-(U5-INPUT_1-Pad2) -> /M1_C
- U5 pad 20: unconnected-(U5-VSS-Pad20) -> +BATT
- U5 pad 3: unconnected-(U5-OUTPUT_1-Pad3) -> /M+1
- U5 pad 4: unconnected-(U5-GND-Pad4) -> GND
- U5 pad 5: unconnected-(U5-GND__1-Pad5) -> GND
- U5 pad 6: unconnected-(U5-GND__2-Pad6) -> GND
- U5 pad 7: unconnected-(U5-GND__3-Pad7) -> GND
- U5 pad 8: unconnected-(U5-OUTPUT_2-Pad8) -> /M-1
- U5 pad 9: unconnected-(U5-INPUT_2-Pad9) -> /M1_CC
Other:
- board outline added: 197.6 x 84 mm

Commit message: pcb done
Parts:
- C2, C5, C6: moved to B.Cu
- moved C1 64.1 mm to (229.4, 229.6), turned to 0 degrees
- moved C2 56.2 mm to (229.9, 221.8), turned to 90 degrees
- moved R1 51.5 mm to (223.1, 220.7), turned to 90 degrees
- moved C6 44.8 mm to (251.0, 197.0), turned to 90 degrees
- moved C5 40.7 mm to (248.0, 197.0), turned to 90 degrees
- moved C3 29.3 mm to (247.0, 188.0), turned to 90 degrees
- moved C4 29.3 mm to (244.0, 188.0), turned to 90 degrees
- moved SW1 22.3 mm to (217.3, 220.0), turned to -90 degrees
- moved U1 8.32 mm to (230.0, 224.7)
- moved J3 6.01 mm to (262.3, 209.5)
- moved J2 5.09 mm to (218.2, 234.6), turned to 0 degrees
- moved J1 4.75 mm to (226.5, 234.5), turned to 0 degrees
- moved U4 3.05 mm to (366.5, 186.0)
- moved J6 2.90 mm to (367.3, 219.3)
- moved U3 2.70 mm to (373.8, 201.3)
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Connections:
- U3 pad 1: VCC -> unconnected-(U3-Vin-Pad1)
- U3 pad 2: unconnected-(U3-3V3-Pad2) -> VCC
- U4 pad 6: VCC -> unconnected-(U4-VIN-Pad6)
- U4 pad 7: unconnected-(U4-3V3-Pad7) -> VCC
Routing:
- net /IR_OUT_1: track 0.00 -> 123.2 mm, vias 0 -> 3
- net /IR_OUT_3: track 0.00 -> 120.7 mm, vias 0 -> 4
- net /IR_OUT_5: track 0.00 -> 117.2 mm, vias 0 -> 1
- net /OLED_MOSI: track 0.00 -> 109.6 mm, vias 0 -> 2
- net /IR_OUT_2: track 0.00 -> 104.4 mm, vias 0 -> 2
- net /OLED_MISO: track 0.00 -> 101.4 mm
- net /OLED_SCL: track 0.00 -> 99.4 mm
- net /Gyro_CS: track 0.00 -> 98.7 mm, vias 0 -> 2
- net /IR_OUT_4: track 0.00 -> 93.1 mm, vias 0 -> 2
- net /OLED_CS: track 0.00 -> 73.0 mm
- net /M1_C: track 0.00 -> 71.5 mm, vias 0 -> 2
- net /Gyro_MOSI: track 0.00 -> 64.4 mm
- net /Gyro_SCL: track 0.00 -> 63.8 mm, vias 0 -> 3
- net +BATT: track 0.00 -> 62.8 mm
- net /ENC2_B: track 0.00 -> 60.2 mm, vias 0 -> 3
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- added copper zone on B.Cu, net GND
- added copper zone on F.Cu, net VCC
Other:
- board size 197.6 x 84 mm -> 184 x 84 mm

Commit message: cut the thing in half
forgot to upload this earlier
Parts:
- removed C1, C6: 10uF, Capacitor_SMD:C_0805_2012Metric_Pad1.18x1.45mm_HandSolder
- removed C2: 22uF, Capacitor_SMD:C_0805_2012Metric_Pad1.18x1.45mm_HandSolder
- removed C3, C5: 4.7uF, Capacitor_SMD:C_0805_2012Metric_Pad1.18x1.45mm_HandSolder
- removed C4: 100nF, Capacitor_SMD:C_0805_2012Metric_Pad1.18x1.45mm_HandSolder
- removed H1, H2, H3, H4, H5, H6: MountingHole, MountingHole:MountingHole_2.5mm
- removed H7, H8: MountingHole, MountingHole:MountingHole_2mm
- removed J1, J2: B2B-PH-K-S, B2B_PH_K_S:JST_B2B-PH-K-S
- removed J3, J4: Conn_01x06_Pin, Connector_JST:JST_SH_BM06B-SRSS-TB_1x06-1MP_P1.00mm_Vertical
- removed J5, J6, J7, J8, J9: Conn_01x03_Pin, Connector_PinSocket_2.54mm:PinSocket_1x03_P2.54mm_Horizontal
- removed R1: 10k, Resistor_SMD:R_0805_2012Metric_Pad1.20x1.40mm_HandSolder
- removed SW1: CL-SB-12A-01T, CL_SB_12A_01T:CL-SB-12A-01T_NDC
- removed U1: AZ1117IH-3.3TRG1, AZ1117IH_3_3TRG1:SOT230P700X185-4N
- removed U2: NUCLEO-L476RG, NUCLEO-L476RG:MODULE_NUCLEO-L476RG
- removed U3: ISM330DHCX, Adafruit_ISM330DHCX:ISM330DHCX
- removed U4: SSD1306, Adafruit_SSD1306:SSD1306
- removed U5: L293DD, L293DD:SOIC127P1032X265-20N
Routing:
- net /IR_OUT_1: track 123.2 -> 0.00 mm, vias 3 -> 0
- net /IR_OUT_3: track 120.7 -> 0.00 mm, vias 4 -> 0
- net /IR_OUT_5: track 117.2 -> 0.00 mm, vias 1 -> 0
- net /OLED_MOSI: track 109.6 -> 0.00 mm, vias 2 -> 0
- net /IR_OUT_2: track 104.4 -> 0.00 mm, vias 2 -> 0
- net /OLED_MISO: track 101.4 -> 0.00 mm
- net /OLED_SCL: track 99.4 -> 0.00 mm
- net /Gyro_CS: track 98.7 -> 0.00 mm, vias 2 -> 0
- net /IR_OUT_4: track 93.1 -> 0.00 mm, vias 2 -> 0
- net /OLED_CS: track 73.0 -> 0.00 mm
- net /M1_C: track 71.5 -> 0.00 mm, vias 2 -> 0
- net /Gyro_MOSI: track 64.4 -> 0.00 mm
- net /Gyro_SCL: track 63.8 -> 0.00 mm, vias 3 -> 0
- net +BATT: track 62.8 -> 0.00 mm
- net /ENC2_B: track 60.2 -> 0.00 mm, vias 3 -> 0
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- removed copper zone on B.Cu, net GND
- removed copper zone on F.Cu, net VCC
Other:
- board size 184 x 84 mm -> 96 x 84 mm
